File: d1-relay-module-shield.sch (EAGLE design)
At the start: 5 parts

Commit message: align d1 with edge of relay board and add cutout for jumper
Parts:
- removed JP2: (no value), pinhead:PINHD-1X3
Changed lines of the file:
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@@
 <part name="U$1" library="diy-modules" deviceset="WEMOS-D1-MINI-SHIELD" device=""/>
 <part name="JP1" library="pinhead" library_urn="urn:adsk.eagle:library:325" deviceset="PINHD-1X4" device="" package3d_urn="urn:adsk.eagle:package:22407/2"/>
-<part name="JP2" library="pinhead" library_urn="urn:adsk.eagle:library:325" deviceset="PINHD-1X3" device="" package3d_urn="urn:adsk.eagle:package:22458/2"/>
 <part name="GND1" library="supply1" library_urn="urn:adsk.eagle:library:371" deviceset="GND" device=""/>
 <part name="P+1" library="supply1" library_urn="urn:adsk.eagle:library:371" deviceset="VCC" device=""/>
@@
 <attribute name="VALUE" x="147.32" y="102.87" size="1.778" layer="96" rot="R270"/>
 </instance>
-<instance part="JP2" gate="A" x="109.22" y="96.52" smashed="yes" rot="R270">
-<attribute name="NAME" x="114.935" y="102.87" size="1.778" layer="95" rot="R270"/>
-<attribute name="VALUE" x="101.6" y="102.87" size="1.778" layer="96" rot="R270"/>
-</instance>
 <instance part="GND1" gate="1" x="144.78" y="81.28" smashed="yes">
